File: source/Cheap FOCer 2 60mm.kicad_pcb (KiCad board)
At the start: 2 copper layers, 59.1 x 99.9 mm, 193 parts, among them J1 Conn_01x02, J2 Conn_01x07, J3 Conn_01x03, J4 On/Off, J5 UNUSED MCU PINS, J6 Conn_01x03, P1 MOTOR1, P2 MOTOR1, P3 MOTOR1, P4 HALL/Encoder, P5 SWD, Q1 NCEP60T20, Q2 NCEP60T20, Q3 NCEP60T20, Q4 NCEP60T20, Q5 NCEP60T20, Q6 NCEP60T20, U1 AMS1117-3.3, U2 DRV8301, U3 TP2604-SR, U4 TJA1051T/3/1J, U5 STM32F405RGT6, U6 BMI160, X1 8MHz 10ppm (X50328MSB2GI)

Commit message: renew kicad to v8
Other:
- net class Default removed
